Commit message: Add files via upload

File: summit_description/urdf/base/summit_base.urdf.xacro (robot description, xacro)
@@ -35,7 +35,9 @@
     <color rgba="1.0 1.0 1.0 1.0"/>
   </material>
+  <!--
   <gazebo reference="base_link">
     <material>Gazebo/Orange</material>
   </gazebo>
+  -->
   <gazebo reference="link_left_wheel">
     <material>Gazebo/Blue</material>
@@ -72,5 +74,5 @@
       <origin rpy="0 0 0" xyz="0 0 0"/>
       <geometry>
-         <mesh filename="package://summit_description/meshes/base/true_bae.dae" />
+        <mesh filename="package://summit_description/meshes/base/true_bae.dae" />
       </geometry>
       <material name="blue"/>
@@ -256,23 +258,4 @@
   <!-- Left Wheel link -->
 <!--
-  <link name="hokuyo">
-    <collision>
-      <origin xyz="0 0 0" rpy="0 0 0"/>
-      <geometry>
-    <box size="0.1 0.1 0.1"/>
-      </geometry>
-    </collision>
-    <visual>
-      <origin xyz="0 0 0" rpy="0 0 0"/>
-      <geometry>
-          <mesh filename="package://summit_description/meshes/base/hokuyo.dae" />
-      </geometry>
-    </visual>
-    <inertial>
-      <mass value="1e-5" />
-      <origin xyz="0 0 0" rpy="0 0 0"/>
-      <inertia ixx="1e-6" ixy="0" ixz="0" iyy="1e-6" iyz="0" izz="1e-6" />
-    </inertial>
-  </link>
     -->
   <joint name="base_link_tower_link_joint" type="fixed">
@@ -315,12 +298,4 @@
         <child link="camera"/>
   </joint>
-  <!--
-  <joint name="hokuyo_joint" type="fixed">
-    <axis xyz="0 1 0" />
-    <origin xyz="0 0 .1" rpy="0 0 3.14"/>
-    <parent link="base_link"/>
-    <child link="hokuyo"/>
-  </joint>
--->
   <joint name="hokuyo_bottom_joint" type="fixed">
     <axis xyz="0 1 0" />
@@ -420,9 +395,10 @@
     </sensor>
   </gazebo>
-  <gazebo reference="hokuyo_bottom">
+  <!--
+  < gazebo reference="hokuyo_bottom">
     <sensor type="gpu_ray" name="head_hokuyo_sensor">
       <pose>0 0 0 0 0 0</pose>
       <visualize>true</visualize>
-      <update_rate>20</update_rate>
+      <update_rate>40</update_rate>
       <ray>
         <scan>
@@ -432,4 +408,36 @@
             <min_angle>-1.57</min_angle>
             <max_angle>1.57</max_angle>
+          </horizontal>
+        </scan>
+        <range>
+          <min>0.10</min>
+          <max>30.0</max>
+          <resolution>0.01</resolution>
+        </range>
+        <noise>
+          <type>gaussian</type>
+          <mean>0.0</mean>
+          <stddev>0.01</stddev>
+        </noise>
+      </ray>
+      <plugin name="gazebo_ros_head_hokuyo_controller" filename="libgazebo_ros_gpu_laser.so">
+        <topicName>/scan</topicName>
+        <frameName>hokuyo_bottom</frameName>
+      </plugin>
+    </sensor>
+  </gazebo >
+  -->
+  <gazebo reference="hokuyo_bottom">
+    <sensor type="ray" name="head_hokuyo_sensor">
+      <pose>0 0 0 0 0 0</pose>
+      <visualize>true</visualize>
+      <update_rate>40</update_rate>
+      <ray>
+        <scan>
+          <horizontal>
+            <samples>720</samples>
+            <resolution>1</resolution>
+            <min_angle>-1.570796</min_angle>
+            <max_angle>1.570796</max_angle>
           </horizontal>
         </scan>
@@ -449,5 +457,5 @@
         </noise>
       </ray>
-      <plugin name="gazebo_ros_head_hokuyo_controller" filename="libgazebo_ros_gpu_laser.so">
+      <plugin name="gazebo_ros_head_hokuyo_controller" filename="libgazebo_ros_laser.so">
         <topicName>/mybot/laser/scan_bottom</topicName>
         <frameName>hokuyo_bottom</frameName>
@@ -455,35 +463,4 @@
     </sensor>
   </gazebo>
-   <!-- gazebo reference="hokuyo">
-    <sensor type="gpu_ray" name="head_hokuyo_sensor">
-      <pose>0 0 0 0 0 0</pose>
-      <visualize>false</visualize>
-      <update_rate>40</update_rate>
-      <ray>
-        <scan>
-          <horizontal>
-            <samples>720</samples>
-            <resolution>1</resolution>
-            <min_angle>-2.47</min_angle>
-            <max_angle>2.57</max_angle>
-          </horizontal>
-        </scan>
-        <range>
-          <min>0.10</min>
-          <max>30.0</max>
-          <resolution>0.01</resolution>
-        </range>
-        <noise>
-          <type>gaussian</type>
-          <mean>0.0</mean>
-          <stddev>0.01</stddev>
-        </noise>
-      </ray>
-      <plugin name="gazebo_ros_head_hokuyo_controller" filename="libgazebo_ros_gpu_laser.so">
-        <topicName>/mybot/laser/scan</topicName>
-        <frameName>hokuyo</frameName>
-      </plugin>
-    </sensor>
-  </gazebo -->
   <gazebo>
     <plugin name="omni_steering" filename="libgazebo_ros_planar_move.so">
